File: Kicad PCB/BOARD.kicad_sch (KiCad schematic)
At the start: 5 parts, among them U3 ESP32-S3-WROOM-1

Commit message: Se modifico el esquematico.
Parts:
- removed R1, R2: 220, PCM_Resistor_SMD_AKL:R_0603_1608Metric, symbol EasyEDA:R_0603
Connections:
- net ENTRAD_NPN_1/NPN_OUT renamed ENTRAD_NPN_1/SALIDA_NPN
Other:
- sheet ENTRAD_NPN_1 ports: added ENTRADA_NPN, SALIDA_NPN; removed NPN_IN, NPN_OUT
Changed lines of the file:
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@@
-	(wire
-		(pts
-			(xy 187.96 138.43) (xy 187.96 142.24)
-		)
-		(stroke
-			(width 0)
-			(type default)
-		)
-	)
 	(wire
 		(pts
@@
 	(wire
 		(pts
-			(xy 187.96 128.27) (xy 185.42 128.27)
-		)
-		(stroke
-			(width 0)
-			(type default)
-		)
-	)
-	(wire
-		(pts
 			(xy 266.7 57.15) (xy 270.51 57.15)
 		)
@@
 	(wire
 		(pts
-			(xy 187.96 130.81) (xy 187.96 128.27)
-		)
-		(stroke
-			(width 0)
-			(type default)
-		)
-	)
-	(wire
-		(pts
 			(xy 190.5 64.77) (xy 185.42 64.77)
 		)
@@
 	(wire
 		(pts
-			(xy 185.42 120.65) (xy 187.96 120.65)
-		)
-		(stroke
-			(width 0)
-			(type default)
-		)
-	)
-	(wire
-		(pts
 			(xy 63.5 52.07) (xy 63.5 57.15)
 		)
@@
 	(wire
 		(pts
-			(xy 189.23 142.24) (xy 187.96 142.24)
-		)
-		(stroke
-			(width 0)
-			(type default)
-		)
-	)
-	(wire
-		(pts
 			(xy 185.42 102.87) (xy 238.76 102.87)
-		)
-		(stroke
-			(width 0)
-			(type default)
-		)
-	)
-	(wire
-		(pts
-			(xy 195.58 120.65) (xy 198.12 120.65)
 		)
 		(stroke
@@
 		)
 	)
-	(hierarchical_label "AUX_2"
-		(shape output)
-		(at 198.12 120.65 0)
-		(effects
-			(font
-				(size 1.27 1.27)
-			)
-			(justify left)
-		)
-	)
 	(hierarchical_label "PNP_IN_2"
 		(shape input)
@@
 			)
 			(justify right)
-		)
-	)
-	(hierarchical_label "AUX_1"
-		(shape output)
-		(at 189.23 142.24 0)
-		(effects
-			(font
-				(size 1.27 1.27)
-			)
-			(justify left)
 		)
 	)
@@
 	)
 	(symbol
-		(lib_id "EasyEDA:R_0603")
-		(at 191.77 120.65 90)
-		(mirror x)
-		(unit 1)
-		(exclude_from_sim no)
-		(in_bom yes)
-		(on_board yes)
-		(dnp no)
-		(fields_autoplaced yes)
-		(property "Reference" "R2"
-			(at 191.77 114.3 90)
-			(effects
-				(font
-					(size 1.27 1.27)
-				)
-			)
-		)
-		(property "Value" "220"
-			(at 191.77 116.84 90)
-			(effects
-				(font
-					(size 1.27 1.27)
-				)
-			)
-		)
-		(property "Footprint" "PCM_Resistor_SMD_AKL:R_0603_1608Metric"
-			(at 203.2 120.65 0)
-			(effects
-				(font
-					(size 1.27 1.27)
-				)
-				(hide yes)
-			)
-		)
-		(property "Datasheet" "~"
-			(at 191.77 120.65 0)
-			(effects
-				(font
-					(size 1.27 1.27)
-				)
-				(hide yes)
-			)
-		)
-		(property "Description" "SMD 0603 Chip Resistor, US Symbol, Alternate KiCad Library"
-			(at 191.77 120.65 0)
-			(effects
-				(font
-					(size 1.27 1.27)
-				)
-				(hide yes)
-			)
-		)
-		(pin "1"
-		)
-		(pin "2"
-		)
-		(instances
-			(project "Juana NIVARA"
-				(path "/1db8b63f-56a3-4827-870b-25f376d196ab/4a0bb713-5b78-4270-b323-33ba352e0a8e"
-					(reference "R2")
-					(unit 1)
-				)
-			)
-		)
-	)
-	(symbol
 		(lib_id "EasyEDA:C_0603")
 		(at 50.8 30.48 0)
@@
 	)
 	(symbol
-		(lib_id "EasyEDA:R_0603")
-		(at 187.96 134.62 0)
-		(mirror y)
-		(unit 1)
-		(exclude_from_sim no)
-		(in_bom yes)
-		(on_board yes)
-		(dnp no)
-		(fields_autoplaced yes)
-		(property "Reference" "R1"
-			(at 185.42 133.3499 0)
-			(effects
-				(font
-					(size 1.27 1.27)
-				)
-				(justify left)
-			)
-		)
-		(property "Value" "220"
-			(at 185.42 135.8899 0)
-			(effects
-				(font
-					(size 1.27 1.27)
-				)
-				(justify left)
-			)
-		)
-		(property "Footprint" "PCM_Resistor_SMD_AKL:R_0603_1608Metric"
-			(at 187.96 146.05 0)
-			(effects
-				(font
-					(size 1.27 1.27)
-				)
-				(hide yes)
-			)
-		)
-		(property "Datasheet" "~"
-			(at 187.96 134.62 0)
-			(effects
-				(font
-					(size 1.27 1.27)
-				)
-				(hide yes)
-			)
-		)
-		(property "Description" "SMD 0603 Chip Resistor, US Symbol, Alternate KiCad Library"
-			(at 187.96 134.62 0)
-			(effects
-				(font
-					(size 1.27 1.27)
-				)
-				(hide yes)
-			)
-		)
-		(pin "1"
-		)
-		(pin "2"
-		)
-		(instances
-			(project "Juana NIVARA"
-				(path "/1db8b63f-56a3-4827-870b-25f376d196ab/4a0bb713-5b78-4270-b323-33ba352e0a8e"
-					(reference "R1")
-					(unit 1)
-				)
-			)
-		)
-	)
-	(symbol
 		(lib_id "EasyEDA:C_0603")
 		(at 81.28 30.48 0)
@@
 			)
 		)
-		(pin "NPN_IN" input
+		(pin "ENTRADA_NPN" input
 			(at 35.56 85.09 180)
 			(effects
@@
 			)
 		)
-		(pin "NPN_OUT" input
+		(pin "SALIDA_NPN" input
 			(at 63.5 85.09 0)
 			(effects
