File: Kicad PCB/ENTRAD_NPN_1.kicad_sch (KiCad schematic)
At the start: 5 parts, among them U6 LTV-357T

Commit message: Se modifico el esquematico.
Connections:
- net NPN_IN renamed ENTRADA_NPN
- net NPN_OUT renamed SALIDA_NPN
Changed lines of the file:
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@@
 		)
 	)
-	(hierarchical_label "NPN_IN"
+	(hierarchical_label "ENTRADA_NPN"
 		(shape input)
 		(at 110.49 62.23 180)
@@
 		)
 	)
-	(hierarchical_label "NPN_OUT"
+	(hierarchical_label "SALIDA_NPN"
 		(shape input)
 		(at 149.86 85.09 0)
